File: PCB/SF65.kicad_pcb (KiCad board)
At the start: 2 copper layers, 321.5 x 135.7 mm, 176 parts, among them J1 C165948_-_USB_C_Receptacle_US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, J2 SM02B-SRSS-TB(LF)(SN), Q1 Q_PMOS_GSD, SW1 CAP_STP, SW10 A, SW11 WIN_1.25U, SW12 2, SW13 W, SW14 S, SW15 Z, SW16 L_ALT_1.25U, SW17 L_ALT_1.5U, SW18 3, SW19 E, SW2 ESC, SW20 D, SW21 X, SW22 4, SW23 R, SW24 F, SW25 C, SW26 5, SW27 T, SW28 G, SW29 V, SW3 Tab, SW30 SPC_6.25U, SW31 SPC_7U, SW32 6, SW33 Y, SW34 H, SW35 B, SW36 7, SW37 U, SW38 J, SW39 N, SW4 CAP, SW40 8, SW41 I, SW42 K, SW43 M, SW44 R_ALT_1U, SW45 R_ALT_1.5U, SW46 9, SW47 O, SW48 L, SW49 ,, SW5 L_SHFT, SW50 R_WIN_1U, SW51 R_CTRL_1.5U, SW52 0, SW53 P, SW54 ;, SW55 ., SW56 R_CTRL_1U, SW57 -, SW58 [, SW59 ', SW6 L_CTRL_1.25U, SW60 /, SW61 =, SW62 ], SW63 R_SHFT_1.75U, SW64 LEFT, SW65 R_SHFT_1.5U, SW66 BCKSP, SW67 \, SW68 ENT, SW69 UP, SW7 L_CTRL_1.5U, SW70 DOWN, SW71 ENT_ISO, SW72 Tilde, SW73 Del, SW74 PG_UP, SW75 PG_DWN, SW76 RIGHT, SW8 1, SW9 Q, U1 TP4054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

Commit message: diodes placed
Parts:
- moved D69 410.3 mm to (214.7, 13.5), turned to 180 degrees
- moved D64 399.4 mm to (201.3, 13.5), turned to 180 degrees
- moved D56 375.2 mm to (174.6, 13.5), turned to 180 degrees
- moved D48 370.0 mm to (239.6, 2.13), turned to 180 degrees
- moved D53 368.0 mm to (240.6, 7.80), turned to 180 degrees
- moved D12 366.6 mm to (226.2, 2.13), turned to 180 degrees
- moved D70 365.6 mm to (215.8, 19.1), turned to 180 degrees
- moved D17 364.7 mm to (227.2, 7.80), turned to 180 degrees
- moved D51 364.4 mm to (161.2, 13.5), turned to 180 degrees
- moved D66 363.5 mm to (241.4, 13.5), turned to 180 degrees
- moved D30 362.6 mm to (228.1, 13.5), turned to 180 degrees
- moved D71 361.9 mm to (242.6, 19.1), turned to 180 degrees
- moved D43 361.0 mm to (229.2, 19.1), turned to 180 degrees
- moved D65 354.8 mm to (202.4, 19.1), turned to 180 degrees
- moved D46 353.6 mm to (147.9, 13.5), turned to 180 degrees
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Routing:
- net Net-(D4-Pad2): track 48.3 -> 12.9 mm
- net Net-(D5-Pad2): track 50.8 -> 23.9 mm
- net Net-(D6-Pad2): track 61.5 -> 43.1 mm
- net Net-(D7-Pad2): track 73.6 -> 71.4 mm
Other:
- board size 321.5 x 135.7 mm -> 310.8 x 135.7 mm

Commit message: working on routing, not complete
Parts:
- added J3: SM02B-SRSS-TB(LF)(SN), Connector_PinHeader_2.54mm:PinHeader_1x02_P2.54mm_Vertical, F.Cu at (288.1, 21.2)
- H1, H2, H3, H4, H5, H6: footprint MountingHole:MountingHole_4.3mm_M4 -> MountingHole:MountingHole_2.2mm_M2
- moved H2 409.9 mm to (325.2, 22.0)
- moved H3 405.2 mm to (325.2, -0.47)
- moved D12 196.9 mm to (29.3, 2.13)
- moved D17 196.9 mm to (30.3, 7.80)
- moved D30 196.9 mm to (31.1, 13.5)
- moved D43 196.9 mm to (32.3, 19.1)
- moved H5 162.4 mm to (24.6, -0.07)
- moved H4 140.7 mm to (24.6, 22.1)
- moved R1 40.0 mm to (288.5, 5.58)
- moved R2 36.3 mm to (286.9, 5.58), turned to -90 degrees
- moved D4 16.7 mm to (42.3, 2.13)
- moved D5 16.7 mm to (43.3, 7.80)
- moved D7 16.7 mm to (45.3, 19.1)
- moved D6 16.5 mm to (44.1, 13.5)
- moved D10 16.3 mm to (56.2, 7.80)
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Connections:
- BLE1 pad 1: row0 -> unconnected-(BLE1-Pad1)
- BLE1 pad 10: col0 -> unconnected-(BLE1-Pad10)
- BLE1 pad 15: P0.05 -> unconnected-(BLE1-Pad15)
- BLE1 pad 17: row2 -> unconnected-(BLE1-Pad17)
- BLE1 pad 2: row1 -> unconnected-(BLE1-Pad2)
- BLE1 pad 28: ENCA -> unconnected-(BLE1-Pad28)
- BLE1 pad 30: ENCB -> unconnected-(BLE1-Pad30)
- BLE1 pad 4: col5 -> unconnected-(BLE1-Pad4)
- BLE1 pad 41: row3 -> unconnected-(BLE1-Pad41)
- BLE1 pad 43: row4 -> unconnected-(BLE1-Pad43)
- BLE1 pad 6: col4 -> unconnected-(BLE1-Pad6)
- BLE1 pad 7: col3 -> unconnected-(BLE1-Pad7)
- BLE1 pad 8: col2 -> unconnected-(BLE1-Pad8)
- BLE1 pad 9: col1 -> unconnected-(BLE1-Pad9)
Routing:
- net Net-(D53-Pad2): track 0.00 -> 306.2 mm
- net Net-(D43-Pad2): track 0.00 -> 277.8 mm
- net Net-(D48-Pad2): track 0.00 -> 275.4 mm
- net Net-(D30-Pad2): track 0.00 -> 217.0 mm
- net Net-(D66-Pad2): track 0.00 -> 211.0 mm
- net Net-(D71-Pad2): track 0.00 -> 185.3 mm
- net Net-(D65-Pad2): track 0.00 -> 175.1 mm
- net Net-(D64-Pad2): track 0.00 -> 171.6 mm
- net Net-(D70-Pad2): track 0.00 -> 171.4 mm
- net Net-(D61-Pad2): track 0.00 -> 168.9 mm, vias 0 -> 1
- net Net-(D69-Pad2): track 0.00 -> 163.3 mm
- net Net-(D60-Pad2): track 0.00 -> 160.2 mm
- net Net-(D52-Pad2): track 0.00 -> 153.8 mm
- net Net-(D68-Pad2): track 0.00 -> 150.2 mm
- net Net-(D57-Pad2): track 0.00 -> 149.7 mm
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Other:
- board size 310.8 x 135.7 mm -> 304.8 x 122.6 mm

Commit message: about to swap in raytac module
Parts:
- added C6: 15pF, Capacitor_SMD:C_0603_1608Metric, F.Cu at (238.4, -11.7)
- added C7: 15pF, Capacitor_SMD:C_0603_1608Metric, F.Cu at (244.2, -17.8)
- added J1: C165948_-_USB_C_Receptacle_USB2.0_SMD, Connector_USB:USB_C_Receptacle_HRO_TYPE-C-31-M-12, F.Cu at (246.9, -23.7)
- added RESET1: SW_Push, Button_Switch_SMD:SW_SPST_B3U-1000P, F.Cu at (239.3, -15.1)
- added SWD/C1: Conn_01x04_Female, Connector_PinHeader_2.54mm:PinHeader_1x04_P2.54mm_Vertical, F.Cu at (238.7, -27.2)
- added U3: MDBT50Q-1MV2, RF_Module:Raytac_MDBT50Q, F.Cu at (229.6, -12.3)
- added Y2: 32.768kHz, COBoards:FC-135R_L3.2-W1.5, F.Cu at (255.0, -28.1)
- C1, C2: value 22pF -> 15pF
- moved R4 308.2 mm to (273.5, -5.20)
- moved R3 304.5 mm to (273.5, -6.82)
- moved R5 301.1 mm to (263.2, -9.20)
- moved D1 281.2 mm to (262.4, -6.47)
- moved H1 139.0 mm to (17.4, 47.8)
- moved H6 139.0 mm to (4.25, 56.5)
- moved J3 0.20 mm to (288.1, 21.0)
Connections:
- BLE1 pad 1: unconnected-(BLE1-Pad1) -> Row0
- BLE1 pad 2: unconnected-(BLE1-Pad2) -> Col0
- BLE1 pad 26: RESET -> unconnected-(BLE1-Pad26)
- BLE1 pad 27: VBUS -> unconnected-(BLE1-Pad27)
- BLE1 pad 29: D- -> unconnected-(BLE1-Pad29)
- BLE1 pad 3: BATTERY_MEASURE -> unconnected-(BLE1-Pad3)
- BLE1 pad 31: D+ -> unconnected-(BLE1-Pad31)
- BLE1 pad 37: SWD -> unconnected-(BLE1-Pad37)
- BLE1 pad 39: SWC -> unconnected-(BLE1-Pad39)
- BLE1 pad 4: unconnected-(BLE1-Pad4) -> Col1
- BLE1 pad 5: GND -> unconnected-(BLE1-Pad5)
- BLE1 pad 6: unconnected-(BLE1-Pad6) -> Col2
Routing:
- net Row4: track 0.00 -> 278.0 mm, vias 0 -> 5
- net Row3: track 0.00 -> 271.6 mm, vias 0 -> 15
- net Row2: track 0.00 -> 262.7 mm, vias 0 -> 15
- net Row1: track 0.00 -> 261.0 mm, vias 0 -> 16
- net Col0: track 44.4 -> 277.1 mm, vias 0 -> 1
- net Row0: track 0.00 -> 225.6 mm
- net Col1: track 85.1 -> 296.5 mm, vias 0 -> 1
- net Col2: track 67.0 -> 257.3 mm, vias 0 -> 1
- net Col3: track 67.0 -> 237.3 mm, vias 0 -> 1
- net Col4: track 69.9 -> 220.3 mm, vias 0 -> 1
- net Col5: track 67.0 -> 197.4 mm, vias 0 -> 1
- net Net-(D29-Pad2): track 0.00 -> 128.5 mm
- net Net-(D34-Pad2): track 0.00 -> 123.5 mm
- net Net-(D8-Pad2): track 2.38 -> 125.8 mm, vias 0 -> 1
- net Net-(D25-Pad2): track 0.00 -> 113.0 mm
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Other:
- outline, holes or cut-outs redrawn
